File: projects/OvenController/OvenController.sch (EAGLE design)
At the start: 42 parts, among them Q1 2.5A/30V, Q2 MBT3904DW1T1, U1 MCP73831, U2 ESP-WROOM-32NARROW, U3 AP2112K-3.3V, U4 CP2102N

Commit message: Initial draft of schematic and part way through PCB layout.
Parts:
- removed C19, C6: 4.7uF, SparkFun-Capacitors:4.7UF0603
- removed J2: (no value), SparkFun-Connectors:CONN_12SM_SQ_NO_SILK
- removed J3: (no value), SparkFun-Connectors:QWIIC_CONNECTORJS-1MM
- removed J4: (no value), SparkFun-Connectors:CONN_161X16_SM_SQ_NOSILK
- removed JP2: LiPo, SparkFun-Connectors:CONN_02-JST-2MM-SMT
- removed LOGO4: FOUR_LAYER_WARNING, SparkFun-Aesthetics:FOUR_LAYER_WARNING
- removed Q1: 2.5A/30V, SparkFun-DiscreteSemi:MOSFET-PCHANNELDMG2307L
- removed R6: 2.0k, SparkFun-Resistors:2.0KOHM1/10W5%(0603)
- removed TP1: TEST-POINTTP_15TH_THRU, SparkFun-Connectors:TEST-POINTTP_15TH_THRU
- removed U2: ESP-WROOM-32NARROW, SparkFun-RF:ESP-WROOM-32NARROW
- added BAKE: 5566-2, con-molex:5566-2
- added BTN_CONN: 5566-10, con-molex:5566-10
- added D4, D5, D6, D7: 3A/40V/500mV, SparkFun-DiscreteSemi:DIODE-SCHOTTKY-B340A
- added IC1: ESP32-WROOM-32U, SamacSysImported:ESP32-WROOM-32U
- added K1, K2, K3, K4, K5: EB2-5NU, SamacSysImported:EB2-5NU
- added R5: 604, SparkFun-Resistors:RESISTOR0603
- added U$21, U$22, U$24: SSM6N7002KFU, tew-transistors:SSM6N7002KFU
- D1: value Yellow -> 3A/40V/500mV; device SparkFun-LED:LED-YELLOW0603 -> SparkFun-DiscreteSemi:DIODE-SCHOTTKY-B340A
- R3: value 1K -> 5k; device SparkFun-Resistors:1KOHM-1/10W-1%(0603) -> SparkFun-Resistors:RESISTOR0603
- U1: value MCP73831 -> LTV-816_OPTO_ISOLATOR"; device SparkFun-PowerIC:MCP73831 -> SparkFun-DiscreteSemi:LTV-816_OPTO_ISOLATOR"
Connections:
- removed net 12: J2.5, U2.IO12
- removed net 14: J2.10, U2.IO14
- removed net 15: J2.8, U2.IO15
- removed net 16: J4.14, U2.IO16
- removed net 17: J4.15, U2.IO17
- removed net 2: U2.IO2
- removed net 20: U2.IO20
- removed net 21: J4.16, U2.IO21
- removed net 27: J2.6, U2.IO27
- removed net 32: J2.9, U2.IO32
- removed net 33: J2.7, U2.IO33
- removed net 35: U2.IO35
- removed net A0: J4.5, U2.IO26
- removed net A1: J4.6, U2.IO25
- removed net A2: J4.7, U2.IO34
- removed net A3: J4.8, U2.SENSOR_VN
- removed net A4: J4.9, U2.SENSOR_VP
- removed net A5: J4.10, U2.IO4
- removed net CHG: D1.C, U1.STAT
- removed net MISO: J4.13, U2.IO19
- removed net MOSI: J4.12, U2.IO18
- removed net N$14: R6.2, U1.PROG
- removed net N$17: D1.A, R3.2
- removed net SCK: J4.11, U2.IO5
- removed net SCL: J2.11, J3.4, U2.IO22
- removed net SDA: J2.12, J3.3, U2.IO23
- removed net VIN: C7.1, D2.C, Q1.S, R8.1, U3.IN
- removed net V_BATT: C6.1, J2.1, JP2.1, Q1.D, U1.VBAT
- new net BTN1_1: BTN_CONN-1.S, K1.COM_1
- new net BTN1_2: BTN_CONN-2.S, K1.NO_1
- new net BTN2_1: BTN_CONN-3.S, K2.COM_1
- new net BTN2_2: BTN_CONN-4.S, K2.NO_1
- new net BTN3_1: BTN_CONN-5.S, K3.COM_1
- new net BTN3_2: BTN_CONN-6.S, K3.NO_1
- new net BTN4_1: BTN_CONN-7.S, K4.COM_1
- new net BTN4_2: BTN_CONN-8.S, K4.NO_1
- new net BTN5_1: BTN_CONN-9.S, K5.COM_1
- new net BTN5_2: BTN_CONN-10.S, K5.NO_1
- new net K1_COIL-: D1.A, K1.COIL_-, U$21G$1.D
- new net K1_CTRL: IC1.IO34, U$21G$1.G
- new net K2_COIL-: D4.A, K2.COIL_-, U$22G$1.D
- new net K2_CTRL: IC1.IO35, U$22G$1.G
- new net K3_COIL-: D6.A, K3.COIL_-, U$22G$2.D
- new net K3_CTRL: IC1.IO32, U$22G$2.G
- new net K4_COIL-: D7.A, K4.COIL_-, U$21G$2.D
- new net K4_CTRL: IC1.IO33, U$21G$2.G
- new net K5_COIL-: D5.A, K5.COIL_-, U$24G$1.D
- new net K5_CTRL: IC1.IO25, U$24G$1.G
- new net N$3: C7.1, D2.C, R8.1, U3.IN
- new net N$4: R3.1, U1.4
- new net N$5: R5.1, U1.1
- new net N$6: BAKE-1.S, U1.2
- new net N$7: BAKE-2.S, R5.2
- net 0: now also IC1.IO0; no longer TP1.1, U2.IO0
- net 13: now also IC1.IO13; no longer J2.4, U2.IO13
- net 3.3V: now also IC1.3V3, R3.2; no longer J3.2, J4.2, U2.3V3
- net CHIP_PU: now also IC1.EN; no longer J4.1, U2.EN
- net EN: no longer J2.2
- net GND: now also IC1.GND_1, IC1.GND_2, IC1.GND_3, IC1.GND_4, U$21G$1.S, U$21G$2.S, U$22G$1.S, U$22G$2.S, U$24G$1.S, U$24G$2.G, U$24G$2.S, U1.3; no longer C19.2, C6.2, J3.1, J4.4, JP2.2, R6.1, U1.VSS, U2.GND, U2.GND@1, U2.GND@15, U2.GND@38
- net RX: now also IC1.TXD0; no longer U2.TXD
- net TX: now also IC1.RXD0; no longer U2.RXD
- net V_USB: now also D1.C, D4.C, D5.C, D6.C, D7.C, K1.COIL_+, K2.COIL_+, K3.COIL_+, K4.COIL_+, K5.COIL_+; no longer C19.1, J2.3, Q1.G, R3.1, U1.VIN
Other:
- note added: "Bake Coil Sense"
- note added: "Based on ESP32 Thing Plus"
- note added: "RELAY DRIVES"
- note added: "Relays"
- note added: "Voltage Regulator"
- note removed: "Charge current: I_CHG = 1000 / R_PROG R_PROG=2k : I_CHG=500mA"
- note removed: "Headers"
- note removed: "Lithium-Polymer Battery Charger (1-cell)"
- note removed: "Original ESP32 Thing by Jim Lindblom"
- note removed: "QWIIC Connector"
- note removed: "V_BATT should be a single- cell LiPo battery."
- note removed: "V_USB - 6V MAX V_BATT - Single Cell (4.2V MAX)"
- note removed: "Voltage Regulator and Battery Charger"
- moved on the sheet: R2, R3

Commit message: Updated schematic and semi-final layout.
Parts:
- removed D1, D4, D5, D6, D7: 3A/40V/500mV, SparkFun-DiscreteSemi:DIODE-SCHOTTKY-B340A
- removed FD1, FD2, FD3, FD4: FIDUCIALUFIDUCIAL, SparkFun-Aesthetics:FIDUCIALUFIDUCIAL
- removed FRAME1: FRAME-LEDGER, SparkFun-Aesthetics:FRAME-LEDGER
- removed H1, H2: STAND-OFFTIGHT, SparkFun-Hardware:STAND-OFFTIGHT
- removed K4, K5: EB2-5NU, SamacSysImported:EB2-5NU
- removed LOGO1: SFE_LOGO_FLAME.1_INCH, SparkFun-Aesthetics:SFE_LOGO_FLAME.1_INCH
- removed LOGO2: OSHW-LOGOMINI, SparkFun-Aesthetics:OSHW-LOGOMINI
- removed LOGO3: SFE_LOGO_NAME_FLAME.1_INCH, SparkFun-Aesthetics:SFE_LOGO_NAME_FLAME.1_INCH
- removed U$21, U$22, U$24: SSM6N7002KFU, tew-transistors:SSM6N7002KFU
- added R10, R11, R12, R6, R9: 301, SparkFun-Resistors:RESISTOR0603
- added R13: 300, rcl:R-US_R1210W
- K1, K2, K3: value EB2-5NU -> CPC2030N; device SamacSysImported:EB2-5NU -> SamacSysImported:CPC2030N
- R5: value 604 -> 300; device SparkFun-Resistors:RESISTOR0603 -> rcl:R-US_R1210W
Connections:
- removed net K1_COIL-: D1.A, K1.COIL_-, U$21G$1.D
- removed net K2_COIL-: D4.A, K2.COIL_-, U$22G$1.D
- removed net K3_COIL-: D6.A, K3.COIL_-, U$22G$2.D
- removed net K4_COIL-: D7.A, K4.COIL_-, U$21G$2.D
- removed net K5_COIL-: D5.A, K5.COIL_-, U$24G$1.D
- removed net N$7 (its old number): BAKE-2.S, R5.2
- new net !BAKE_ON: IC1.IO5, R3.1, U1.4
- new net N$11: K2.CONTROL_-_1, R10.2
- new net N$13: K2.CONTROL_-_2, R11.2
- new net N$14: K3.CONTROL_-_1, R12.2
- new net N$5: R13.1, R5.2
- new net N$8: K1.CONTROL_-_1, R6.2
- new net N$9: K1.CONTROL_-_2, R9.2
- net BTN1_1: now also K1.LOAD_1_1; no longer K1.COM_1
- net BTN1_2: now also K1.LOAD_1_2; no longer K1.NO_1
- net BTN2_1: now also K1.LOAD_2_1; no longer K2.COM_1
- net BTN2_2: now also K1.LOAD_2_2; no longer K2.NO_1
- net BTN3_1: now also K2.LOAD_1_1; no longer K3.COM_1
- net BTN3_2: now also K2.LOAD_1_2; no longer K3.NO_1
- net BTN4_1: now also K2.LOAD_2_1; no longer K4.COM_1
- net BTN4_2: now also K2.LOAD_2_2; no longer K4.NO_1
- net BTN5_1: now also K3.LOAD_1_1; no longer K5.COM_1
- net BTN5_2: now also K3.LOAD_1_2; no longer K5.NO_1
- net GND: now also R10.1, R11.1, R12.1, R6.1, R9.1; no longer U$21G$1.S, U$21G$2.S, U$22G$1.S, U$22G$2.S, U$24G$1.S, U$24G$2.G, U$24G$2.S
- net K1_CTRL: now also K1.CONTROL_+_1; no longer U$21G$1.G
- net K2_CTRL: now also K1.CONTROL_+_2; no longer U$22G$1.G
- net K3_CTRL: now also K2.CONTROL_+_1; no longer U$22G$2.G
- net K4_CTRL: now also K2.CONTROL_+_2; no longer U$21G$2.G
- net K5_CTRL: now also K3.CONTROL_+_1; no longer U$24G$1.G
- net N$4: now also BAKE-2.S, R13.2; no longer R3.1, U1.4
- net V_USB: no longer D1.C, D4.C, D5.C, D6.C, D7.C, K1.COIL_+, K2.COIL_+, K3.COIL_+, K4.COIL_+, K5.COIL_+
Other:
- note removed: "RELAY DRIVES"
- moved on the sheet: BAKE-1, BAKE-2, R5

Commit message: OvenController v1.0 as ordered.
Parts:
- C10: device SparkFun-Capacitors:1.0UF-0402-16V-10% -> SparkFun-Capacitors:1.0UF-0603-16V-10%-X7R
- J5: value (none) -> UJ2-MIBH2-4-SMT-TR; device SparkFun-Connectors:USB_MICRO-B_HALF_PTH_MILL -> tew-connectors:UJ2-MIBH2-4-SMT-TR
- R8: value 100K -> 100k; device SparkFun-Resistors:100KOHM-0402-1/16W-1% -> SparkFun-Resistors:100KOHM-0603-1/10W-1%
Connections:
- net GND: now also J5.SHIELD
Changed lines of the file:
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@@
 <part name="GND15" library="SparkFun-Aesthetics" deviceset="GND" device=""/>
 <part name="C7" library="SparkFun-Capacitors" deviceset="1.0UF" device="-0603-16V-10%-X7R" value="1.0uF"/>
-<part name="C10" library="SparkFun-Capacitors" deviceset="1.0UF" device="-0402-16V-10%" value="1.0uF"/>
+<part name="C10" library="SparkFun-Capacitors" deviceset="1.0UF" device="-0603-16V-10%-X7R" value="1.0uF"/>
 <part name="GND21" library="SparkFun-Aesthetics" deviceset="GND" device=""/>
 <part name="GND14" library="SparkFun-Aesthetics" deviceset="GND" device=""/>
@@
 <part name="R4" library="SparkFun-Resistors" deviceset="1KOHM" device="-0603-1/10W-1%" value="1k"/>
 <part name="GND5" library="SparkFun-Aesthetics" deviceset="GND" device=""/>
-<part name="R8" library="SparkFun-Resistors" deviceset="100KOHM" device="-0402-1/16W-1%" value="100K"/>
+<part name="R8" library="SparkFun-Resistors" deviceset="100KOHM" device="-0603-1/10W-1%" value="100k"/>
 <part name="S2" library="SparkFun-Switches" deviceset="MOMENTARY-SWITCH-SPST-2" device="-SMD-4.6X2.8MM" value="0"/>
 <part name="GND10" library="SparkFun-Aesthetics" deviceset="GND" device=""/>
-<part name="J5" library="SparkFun-Connectors" deviceset="USB_MICRO-B" device="_HALF_PTH_MILL"/>
+<part name="J5" library="tew-connectors" deviceset="UJ2-MIBH2-4-SMT-TR" device=""/>
 <part name="IC1" library="SamacSysImported" deviceset="ESP32-WROOM-32U" device=""/>
 <part name="GND8" library="SparkFun-Aesthetics" deviceset="GND" device=""/>
@@
 <attribute name="VALUE" x="284.48" y="76.2" size="1.778" layer="96"/>
 </instance>
-<instance part="J5" gate="J1" x="294.64" y="238.76" smashed="yes">
+<instance part="J5" gate="G$1" x="294.64" y="238.76" smashed="yes">
 <attribute name="VALUE" x="292.1" y="228.854" size="1.778" layer="96" font="vector" rot="MR180" align="top-left"/>
 <attribute name="NAME" x="292.1" y="249.174" size="1.778" layer="95" font="vector"/>
@@
 <segment>
 <pinref part="GND26" gate="1" pin="GND"/>
-<wire x1="322.58" y1="236.22" x2="322.58" y2="218.44" width="0.1524" layer="91"/>
-<wire x1="322.58" y1="236.22" x2="312.42" y2="236.22" width="0.1524" layer="91"/>
-<pinref part="J5" gate="J1" pin="GND"/>
-<wire x1="312.42" y1="236.22" x2="299.72" y2="236.22" width="0.1524" layer="91"/>
+<wire x1="322.58" y1="236.22" x2="322.58" y2="233.68" width="0.1524" layer="91"/>
+<wire x1="322.58" y1="233.68" x2="322.58" y2="218.44" width="0.1524" layer="91"/>
+<pinref part="J5" gate="G$1" pin="GND"/>
+<wire x1="322.58" y1="236.22" x2="299.72" y2="236.22" width="0.1524" layer="91"/>
+<pinref part="J5" gate="G$1" pin="SHIELD"/>
+<wire x1="299.72" y1="233.68" x2="322.58" y2="233.68" width="0.1524" layer="91"/>
+<junction x="322.58" y="233.68"/>
 </segment>
 <segment>
@@
 <wire x1="335.28" y1="231.14" x2="335.28" y2="233.68" width="0.1524" layer="91"/>
 <junction x="335.28" y="233.68"/>
-<pinref part="J5" gate="J1" pin="VBUS"/>
+<pinref part="J5" gate="G$1" pin="VBUS"/>
 <wire x1="312.42" y1="246.38" x2="299.72" y2="246.38" width="0.1524" layer="91"/>
 </segment>
@@
 <pinref part="U4" gate="G$1" pin="D-"/>
 <wire x1="327.66" y1="241.3" x2="345.44" y2="241.3" width="0.1524" layer="91"/>
-<pinref part="J5" gate="J1" pin="D-"/>
+<pinref part="J5" gate="G$1" pin="D-"/>
 <wire x1="312.42" y1="243.84" x2="299.72" y2="243.84" width="0.1524" layer="91"/>
 </segment>
@@
 <pinref part="U4" gate="G$1" pin="D+"/>
 <wire x1="327.66" y1="243.84" x2="345.44" y2="243.84" width="0.1524" layer="91"/>
-<pinref part="J5" gate="J1" pin="D+"/>
+<pinref part="J5" gate="G$1" pin="D+"/>
 <wire x1="312.42" y1="241.3" x2="299.72" y2="241.3" width="0.1524" layer="91"/>
 </segment>
@@
 <wire x1="396.24" y1="71.12" x2="401.32" y2="71.12" width="0.1524" layer="91"/>
 <label x="401.32" y="71.12" size="1.27" layer="95" xref="yes"/>
-</segment>
-<segment>
+<junction x="396.24" y="71.12"/>
+</segment>
+<segment>
